Commit message: fix: change robot size / wheel placement

File: description/lidar.xacro (robot description, xacro)
@@ -4,5 +4,5 @@
         <parent link="chassis"/>
         <child link="laser_frame"/>
-        <origin xyz="0.122 0 0.212" rpy="0 0 0"/>
+        <origin xyz="0.436 0 0.212" rpy="0 0 0"/>
     </joint>
     <link name="laser_frame">
@@ -25,5 +25,5 @@
             </geometry>
         </collision>
-        <xacro:inertial_cylinder mass="0.1" length="0.04" radius="0.05">
+        <xacro:inertial_cylinder mass="0.0" length="0.04" radius="0.05">
             <origin xyz="0 0 0" rpy="0 0 0"/>
         </xacro:inertial_cylinder>

File: description/robot_core.xacro (robot description, xacro)
@@ -2,10 +2,10 @@
 <robot xmlns:xacro="http://www.ros.org/wiki/xacro" >
     <xacro:include filename="inertial_macros.xacro"/>
-    <xacro:property name="chassis_length" value="0.5"/>
-    <xacro:property name="chassis_width" value="0.362"/>
+    <xacro:property name="chassis_length" value="0.486"/>
+    <xacro:property name="chassis_width" value="0.265"/>
     <xacro:property name="chassis_height" value="0.138"/>
     <xacro:property name="chassis_mass" value="1.0"/>
     <xacro:property name="wheel_radius" value="0.051"/>
-    <xacro:property name="wheel_thickness" value="0.026"/>
+    <xacro:property name="wheel_thickness" value="0.038"/>
     <xacro:property name="wheel_mass" value="0.05"/>
     <xacro:property name="wheel_offset_x" value="0.25"/>
@@ -15,5 +15,5 @@
     <xacro:property name="caster_wheel_mass" value="0.01"/>
     <xacro:property name="caster_wheel_offset_x" value="0.075"/>
-    <!-- <xacro:property name="caster_wheel_offset_x_2" value="0.425"/> -->
+    <xacro:property name="caster_wheel_offset_x_2" value="0.425"/>
     <xacro:property name="caster_wheel_offset_z" value="${wheel_offset_z - wheel_radius + caster_wheel_radius}"/>
     <material name="white">
@@ -128,9 +128,4 @@
         <origin xyz="${caster_wheel_offset_x} 0 ${caster_wheel_offset_z}"/>
     </joint>
-    <!-- <joint name="caster_wheel_joint2" type="fixed">
-        <parent link="chassis"/>
-        <child link="caster_wheel_2"/>
-        <origin xyz="${caster_wheel_offset_x_2} 0 ${caster_wheel_offset_z}"/>
-    </joint> -->
     <link name="caster_wheel">
         <visual>
@@ -149,20 +144,4 @@
         </xacro:inertial_sphere>
     </link>
-    <!-- <link name="caster_wheel_2">
-        <visual>
-            <geometry>
-                <sphere radius="${caster_wheel_radius}"/>
-            </geometry>
-            <material name="white"/>
-        </visual>
-        <collision>
-            <geometry>
-                <sphere radius="${caster_wheel_radius}"/>
-            </geometry>
-        </collision>
-        <xacro:inertial_sphere mass="${caster_wheel_mass}" radius="${caster_wheel_radius}">
-            <origin xyz="0 0 0" rpy="0 0 0"/>
-        </xacro:inertial_sphere>
-    </link> -->
     <gazebo reference="caster_wheel">
         <material>Gazebo/White</material>
@@ -170,8 +149,3 @@
         <mu2 value="0.001"/>
     </gazebo>
-    <!-- <gazebo reference="caster_wheel_2">
-        <material>Gazebo/White</material>
-        <mu1 value="0.001"/>
-        <mu2 value="0.001"/>
-    </gazebo> -->
 </robot>
