Commit message: fix: finetune nav2 params

File: description/robot_core.xacro (robot description, xacro)
@@ -3,5 +3,5 @@
     <xacro:include filename="inertial_macros.xacro"/>
     <xacro:property name="chassis_length" value="0.486"/>
-    <xacro:property name="chassis_width" value="0.265"/>
+    <xacro:property name="chassis_width" value="0.324"/>
     <xacro:property name="chassis_height" value="0.138"/>
     <xacro:property name="chassis_mass" value="1.0"/>

Commit message: fix: adapt nav params

File: description/robot_core.xacro (robot description, xacro)
@@ -13,4 +13,5 @@
     <xacro:property name="wheel_offset_z" value="0.01"/>
     <xacro:property name="caster_wheel_radius" value="0.01"/>
+    <xacro:property name="caster_wheel_radius_2" value="0.009"/>
     <xacro:property name="caster_wheel_mass" value="0.01"/>
     <xacro:property name="caster_wheel_offset_x" value="0.075"/>
@@ -128,4 +129,9 @@
         <origin xyz="${caster_wheel_offset_x} 0 ${caster_wheel_offset_z}"/>
     </joint>
+    <joint name="caster_wheel_joint_2" type="fixed">
+        <parent link="chassis"/>
+        <child link="caster_wheel_2"/>
+        <origin xyz="${caster_wheel_offset_x_2} 0 ${caster_wheel_offset_z}"/>
+    </joint>
     <link name="caster_wheel">
         <visual>
@@ -144,4 +150,20 @@
         </xacro:inertial_sphere>
     </link>
+    <link name="caster_wheel_2">
+        <visual>
+            <geometry>
+                <sphere radius="${caster_wheel_radius_2}"/>
+            </geometry>
+            <material name="white"/>
+        </visual>
+        <collision>
+            <geometry>
+                <sphere radius="${caster_wheel_radius_2}"/>
+            </geometry>
+        </collision>
+        <xacro:inertial_sphere mass="${caster_wheel_mass}" radius="${caster_wheel_radius_2}">
+            <origin xyz="0 0 0" rpy="0 0 0"/>
+        </xacro:inertial_sphere>
+    </link>
     <gazebo reference="caster_wheel">
         <material>Gazebo/White</material>
@@ -149,3 +171,8 @@
         <mu2 value="0.001"/>
     </gazebo>
+    <gazebo reference="caster_wheel_2">
+        <material>Gazebo/White</material>
+        <mu1 value="0.001"/>
+        <mu2 value="0.001"/>
+    </gazebo>
 </robot>
