Commit message: update for new robot + sim

File: description/gazebo_control.xacro (robot description, xacro)
@@ -6,6 +6,6 @@
             <left_joint>left_wheel_joint</left_joint>
             <right_joint>right_wheel_joint</right_joint>
-            <wheel_separation>0.288</wheel_separation>
-            <wheel_diameter>0.06</wheel_diameter>
+            <wheel_separation>0.362</wheel_separation>
+            <wheel_diameter>0.051</wheel_diameter>
             <!-- Limits -->
             <max_wheel_torque>200</max_wheel_torque>

File: description/robot_core.xacro (robot description, xacro)
@@ -2,17 +2,18 @@
 <robot xmlns:xacro="http://www.ros.org/wiki/xacro" >
     <xacro:include filename="inertial_macros.xacro"/>
-    <xacro:property name="chassis_length" value="0.335"/>
-    <xacro:property name="chassis_width" value="0.265"/>
+    <xacro:property name="chassis_length" value="0.5"/>
+    <xacro:property name="chassis_width" value="0.362"/>
     <xacro:property name="chassis_height" value="0.138"/>
     <xacro:property name="chassis_mass" value="1.0"/>
-    <xacro:property name="wheel_radius" value="0.06"/>
+    <xacro:property name="wheel_radius" value="0.051"/>
     <xacro:property name="wheel_thickness" value="0.026"/>
     <xacro:property name="wheel_mass" value="0.05"/>
-    <xacro:property name="wheel_offset_x" value="0.288"/>
-    <xacro:property name="wheel_offset_y" value="0.1485"/>
+    <xacro:property name="wheel_offset_x" value="0.25"/>
+    <xacro:property name="wheel_offset_y" value="0.181"/>
     <xacro:property name="wheel_offset_z" value="0.01"/>
     <xacro:property name="caster_wheel_radius" value="0.01"/>
     <xacro:property name="caster_wheel_mass" value="0.01"/>
     <xacro:property name="caster_wheel_offset_x" value="0.075"/>
+    <!-- <xacro:property name="caster_wheel_offset_x_2" value="0.425"/> -->
     <xacro:property name="caster_wheel_offset_z" value="${wheel_offset_z - wheel_radius + caster_wheel_radius}"/>
     <material name="white">
@@ -127,4 +128,9 @@
         <origin xyz="${caster_wheel_offset_x} 0 ${caster_wheel_offset_z}"/>
     </joint>
+    <!-- <joint name="caster_wheel_joint2" type="fixed">
+        <parent link="chassis"/>
+        <child link="caster_wheel_2"/>
+        <origin xyz="${caster_wheel_offset_x_2} 0 ${caster_wheel_offset_z}"/>
+    </joint> -->
     <link name="caster_wheel">
         <visual>
@@ -143,4 +149,20 @@
         </xacro:inertial_sphere>
     </link>
+    <!-- <link name="caster_wheel_2">
+        <visual>
+            <geometry>
+                <sphere radius="${caster_wheel_radius}"/>
+            </geometry>
+            <material name="white"/>
+        </visual>
+        <collision>
+            <geometry>
+                <sphere radius="${caster_wheel_radius}"/>
+            </geometry>
+        </collision>
+        <xacro:inertial_sphere mass="${caster_wheel_mass}" radius="${caster_wheel_radius}">
+            <origin xyz="0 0 0" rpy="0 0 0"/>
+        </xacro:inertial_sphere>
+    </link> -->
     <gazebo reference="caster_wheel">
         <material>Gazebo/White</material>
@@ -148,3 +170,8 @@
         <mu2 value="0.001"/>
     </gazebo>
+    <!-- <gazebo reference="caster_wheel_2">
+        <material>Gazebo/White</material>
+        <mu1 value="0.001"/>
+        <mu2 value="0.001"/>
+    </gazebo> -->
 </robot>

Commit message: feat: URDF robot

File: description/gazebo_control.xacro (robot description, xacro)
@@ -7,5 +7,6 @@
             <right_joint>right_wheel_joint</right_joint>
             <wheel_separation>0.362</wheel_separation>
-            <wheel_diameter>0.051</wheel_diameter>
+            <!-- <wheel_diameter>0.051</wheel_diameter> -->
+            <wheel_diameter>0.51</wheel_diameter>
             <!-- Limits -->
             <max_wheel_torque>200</max_wheel_torque>

File: description/robot.urdf.xacro (robot description, xacro)
@@ -3,5 +3,6 @@
     <xacro:arg name="use_ros2_control" default="true"/>
     <xacro:arg name="sim_mode" default="false"/>
-    <xacro:include filename="robot_core.xacro" />
+    <!-- <xacro:include filename="robot_core.xacro" /> -->
+    <xacro:include filename="urdf_blockbuster.xacro" />
     <xacro:if value="$(arg use_ros2_control)">
         <xacro:include filename="ros2_control.xacro" />
@@ -10,7 +11,5 @@
         <xacro:include filename="gazebo_control.xacro" />
     </xacro:unless>
-    <xacro:include filename="lidar.xacro" />
-    <!-- <xacro:include filename="camera.xacro" /> -->
-    <!-- <xacro:include filename="depth_camera.xacro" /> -->
-    <xacro:include filename="face.xacro" />
+    <xacro:include filename="$(find articubot_one)/description/depthai_macro.urdf.xacro"/>
+    <xacro:depthai_camera camera_name = "oak" parent = "base_link" camera_model = "OAK-D-LITE" base_frame = "oak-d_frame" cam_pos_x = "0.2616" cam_pos_y = "-0.0001" cam_pos_z = "0.20" cam_roll = "0" cam_pitch = "0.785" cam_yaw = "0"/>
 </robot>

File: description/robot_core.xacro (robot description, xacro)
@@ -71,57 +71,48 @@
         <material>Gazebo/Orange</material>
     </gazebo>
-    <!-- LEFT WHEEL LINK -->
     <joint name="left_wheel_joint" type="continuous">
-        <parent link="base_link"/>
-        <child link="left_wheel"/>
-        <origin xyz="0 ${wheel_offset_y} 0" rpy="-${pi/2} 0 0" />
-        <axis xyz="0 0 1"/>
-    </joint>
-    <link name="left_wheel">
-        <visual>
-            <geometry>
-                <cylinder radius="${wheel_radius}" length="${wheel_thickness}"/>
-            </geometry>
-            <material name="blue"/>
-        </visual>
-        <collision>
-            <geometry>
-                <sphere radius="${wheel_radius}"/>
-            </geometry>
-        </collision>
-        <xacro:inertial_cylinder mass="${wheel_mass}" length="${wheel_thickness}" radius="${wheel_radius}">
-            <origin xyz="0 0 0" rpy="0 0 0"/>
-        </xacro:inertial_cylinder>
-    </link>
-    <gazebo reference="left_wheel">
-        <material>Gazebo/Blue</material>
-    </gazebo>
-    <!-- RIGHT WHEEL LINK -->
+        <origin xyz="0.0 0.181 0" rpy="1.57 0 0"/>
+        <parent link="base_link"/>
+        <child link="Left_Wheel_1"/>
+        <axis xyz="0.0 0.0 -1.0"/>
+    </joint>
     <joint name="right_wheel_joint" type="continuous">
-        <parent link="base_link"/>
-        <child link="right_wheel"/>
-        <origin xyz="0 ${-wheel_offset_y} 0" rpy="${pi/2} 0 0" />
-        <axis xyz="0 0 -1"/>
-    </joint>
-    <link name="right_wheel">
-        <visual>
-            <geometry>
-                <cylinder radius="${wheel_radius}" length="${wheel_thickness}"/>
-            </geometry>
-            <material name="blue"/>
-        </visual>
-        <collision>
-            <geometry>
-                <sphere radius="${wheel_radius}"/>
-            </geometry>
-        </collision>
-        <xacro:inertial_cylinder mass="${wheel_mass}" length="${wheel_thickness}" radius="${wheel_radius}">
-            <origin xyz="0 0 0" rpy="0 0 0"/>
-        </xacro:inertial_cylinder>
-    </link>
-    <gazebo reference="right_wheel">
-        <material>Gazebo/Blue</material>
-    </gazebo>
-    <!-- CASTER WHEEL LINK -->
+        <origin xyz="0.0 -0.181 0" rpy="1.57 0 0"/>
+        <parent link="base_link"/>
+        <child link="Right_Wheel_1"/>
+        <axis xyz="0.0 0.0 -1.0"/>
+    </joint>
+    <link name="Left_Wheel_1">
+        <visual>
+            <geometry>
+                <cylinder radius="0.051" length="0.04"/>
+            </geometry>
+        </visual>
+        <collision>
+            <geometry>
+                <sphere radius="0.051"/>
+            </geometry>
+        </collision>
+        <inertial>
+            <mass value="0.04021467988426049"/>
+            <inertia ixx="4e-05" iyy="7e-05" izz="4e-05" ixy="-0.0" iyz="0.0" ixz="0.0"/>
+        </inertial>
+    </link>
+    <link name="Right_Wheel_1">
+        <visual>
+            <geometry>
+                <cylinder radius="0.051" length="0.04"/>
+            </geometry>
+        </visual>
+        <collision>
+            <geometry>
+                <sphere radius="0.051"/>
+            </geometry>
+        </collision>
+        <inertial>
+            <mass value="0.04021467988426049"/>
+            <inertia ixx="4e-05" iyy="7e-05" izz="4e-05" ixy="-0.0" iyz="0.0" ixz="0.0"/>
+        </inertial>
+    </link>
     <joint name="caster_wheel_joint" type="fixed">
         <parent link="chassis"/>
@@ -176,3 +167,106 @@
         <mu2 value="0.001"/>
     </gazebo>
+    <link name="laser_frame">
+    <inertial>
+        <origin xyz="0.01251420264635135 -0.0003851719055572161 -0.019070722094365028" rpy="0 0 0"/>
+        <mass value="0.05"/>
+        <inertia ixx="0.000237" iyy="0.00047" izz="0.000552" ixy="-5e-06" iyz="2e-06" ixz="4.6e-05"/>
+    </inertial>
+    <visual>
+        <origin xyz="-0.104 0.0 -0.2005" rpy="0 0 0"/>
+        <geometry>
+        <mesh filename="file://$(find articubot_one)/meshes/Lidar_1.stl" scale="0.001 0.001 0.001"/>
+        </geometry>
+        <material name="silver"/>
+    </visual>
+    <collision>
+        <origin xyz="-0.104 0.0 -0.2005" rpy="0 0 0"/>
+        <geometry>
+        <mesh filename="file://$(find articubot_one)/meshes/Lidar_1.stl" scale="0.001 0.001 0.001"/>
+        </geometry>
+    </collision>
+    </link>
+    <link name="Stereo_Cam_v1_1">
+    <inertial>
+        <origin xyz="0.015712531986192935 -0.0029261208772013163 -0.003676080873827342" rpy="0 0 0"/>
+        <mass value="0.05"/>
+        <inertia ixx="0.000131" iyy="1.9e-05" izz="0.000127" ixy="0.0" iyz="0.0" ixz="1e-06"/>
+    </inertial>
+    <visual>
+        <origin xyz="-0.236 -0.003 -0.208" rpy="0 0 0"/>
+        <geometry>
+        <mesh filename="file://$(find articubot_one)/meshes/Stereo_Cam_v1_1.stl" scale="0.001 0.001 0.001"/>
+        </geometry>
+        <material name="silver"/>
+    </visual>
+    <collision>
+        <origin xyz="-0.236 -0.003 -0.208" rpy="0 0 0"/>
+        <geometry>
+        <mesh filename="file://$(find articubot_one)/meshes/Stereo_Cam_v1_1.stl" scale="0.001 0.001 0.001"/>
+        </geometry>
+    </collision>
+    </link>
+    <link name="Cam_Window_v1_1">
+    <inertial>
+        <origin xyz="0.00030096983363708807 9.047531604119974e-16 -0.00505688016766781" rpy="0 0 0"/>
+        <mass value="0.01017492506663265"/>
+        <inertia ixx="7e-06" iyy="1e-06" izz="6e-06" ixy="0.0" iyz="0.0" ixz="-0.0"/>
+    </inertial>
+    <visual>
+        <origin xyz="-0.2616 0.0001 -0.208539" rpy="0 0 0"/>
+        <geometry>
+        <mesh filename="file://$(find articubot_one)/meshes/Cam_Window_v1_1.stl" scale="0.001 0.001 0.001"/>
+        </geometry>
+        <material name="silver"/>
+    </visual>
+    <collision>
+        <origin xyz="-0.2616 0.0001 -0.208539" rpy="0 0 0"/>
+        <geometry>
+        <mesh filename="file://$(find articubot_one)/meshes/Cam_Window_v1_1.stl" scale="0.001 0.001 0.001"/>
+        </geometry>
+    </collision>
+    </link>
+    <joint name="laser_joint" type="fixed">
+        <origin xyz="0.121 0.0 0.2358" rpy="0 0 0"/>
+        <parent link="base_link"/>
+        <child link="laser_frame"/>
+    </joint>
+    <joint name="Stereo Cam" type="fixed">
+        <origin xyz="0.236 0.003 0.208" rpy="0 0.785 0"/>
+        <parent link="base_link"/>
+        <child link="Stereo_Cam_v1_1"/>
+    </joint>
+    <joint name="Cam Window" type="fixed">
+        <origin xyz="0.0256 -0.0031 0.000539" rpy="0 0 0"/>
+        <parent link="Stereo_Cam_v1_1"/>
+        <child link="Cam_Window_v1_1"/>
+    </joint>
+    <gazebo reference="laser_frame">
+        <material>Gazebo/Black</material>
+        <sensor name="laser" type="ray">
+            <pose> 0 0 0 0 0 0 </pose>
+            <visualize>false</visualize>
+            <update_rate>10</update_rate>
+            <ray>
+                <scan>
+                    <horizontal>
+                        <samples>360</samples>
+                        <min_angle>-3.14</min_angle>
+                        <max_angle>3.14</max_angle>
+                    </horizontal>
+                </scan>
+                <range>
+                    <min>0.3</min>
+                    <max>12</max>
+                </range>
+            </ray>
+            <plugin name="laser_controller" filename="libgazebo_ros_ray_sensor.so">
+                <ros>
+                    <argument>~/out:=scan</argument>
+                </ros>
+                <output_type>sensor_msgs/LaserScan</output_type>
+                <frame_name>laser_frame</frame_name>
+            </plugin>
+        </sensor>
+    </gazebo>
 </robot>
