Commit message: feat: adding strorage servo

File: description/depthai_macro.urdf.xacro (robot description, xacro)
@@ -31,4 +31,27 @@
                 <child link="${camera_name}_rgb_camera_optical_frame"/>
             </joint>
+            <!-- <gazebo reference="${camera_name}_rgb_camera_frame">
+                <material>Gazebo/Black</material>
+                <sensor name="camera" type="camera">
+                    <pose> 0 0 0 0 0 0 </pose>
+                    <visualize>true</visualize>
+                    <update_rate>10</update_rate>
+                    <camera>
+                        <horizontal_fov>1.089</horizontal_fov>
+                        <image>
+                            <format>R8G8B8</format>
+                            <width>640</width>
+                            <height>480</height>
+                        </image>
+                        <clip>
+                            <near>0.05</near>
+                            <far>8.0</far>
+                        </clip>
+                    </camera>
+                    <plugin name="camera_controller" filename="libgazebo_ros_camera.so">
+                        <frame_name>camera_link_optical</frame_name>
+                    </plugin>
+                </sensor>
+            </gazebo> -->
         </xacro:unless>
         <xacro:unless value="${model in ['OAK-D-LR']}">

File: description/ros2_control.xacro (robot description, xacro)
@@ -7,4 +7,5 @@
                 <param name="left_wheel_name">left_wheel_joint</param>
                 <param name="right_wheel_name">right_wheel_joint</param>
+                <param name="left_servo_name">storage_joint</param>
                 <param name="loop_rate">30</param>
                 <param name="device">/dev/ttyACM0</param>
@@ -29,4 +30,12 @@
                     <param name="min">-10</param>
                     <param name="max">10</param>
+                </command_interface>
+                <state_interface name="position"/>
+                <state_interface name="velocity"/>
+            </joint>
+            <joint name="storage_joint">
+                <command_interface name="velocity">
+                    <param name="min">-5</param>
+                    <param name="max">5</param>
                 </command_interface>
                 <state_interface name="position"/>
@@ -56,4 +65,12 @@
                 <state_interface name="position"/>
             </joint>
+            <joint name="storage_joint">
+                <command_interface name="velocity">
+                    <param name="min">-5</param>
+                    <param name="max">5</param>
+                </command_interface>
+                <state_interface name="velocity"/>
+                <state_interface name="position"/>
+            </joint>
         </ros2_control>
     </xacro:if>

File: description/urdf_blockbuster.xacro (robot description, xacro)
@@ -267,4 +267,25 @@
   <child link="laser_frame"/>
 </joint>
+<joint name="storage_joint" type="continuous">
+  <origin xyz="-0.20 0.16 0.20" rpy="1.57 0 0"/>
+  <parent link="base_link"/>
+  <child link="servo_frame"/>
+</joint>
+<link name="servo_frame">
+    <visual>
+        <geometry>
+            <cylinder radius="0.01" length="0.005"/>
+        </geometry>
+    </visual>
+    <collision>
+        <geometry>
+            <sphere radius="0.051"/>
+        </geometry>
+    </collision>
+    <inertial>
+        <mass value="0.04021467988426049"/>
+        <inertia ixx="4e-05" iyy="7e-05" izz="4e-05" ixy="-0.0" iyz="0.0" ixz="0.0"/>
+    </inertial>
+</link>
 <gazebo reference="laser_frame">
     <material>Gazebo/Black</material>
