Commit message: fix: correction urdf

File: description/urdf_blockbuster.xacro (robot description, xacro)
@@ -268,5 +268,5 @@
 </joint>
 <joint name="storage_joint" type="continuous">
-  <origin xyz="-0.20 0.16 0.20" rpy="1.57 0 0"/>
+  <origin xyz="-0.20 0.13 0.20" rpy="1.57 0 0"/>
   <parent link="base_link"/>
   <child link="servo_frame"/>
