Commit message: feat: changing name to blockbuster_core

File: description/base_macro.urdf.xacro (robot description, xacro)
@@ -19,5 +19,5 @@
                 <origin xyz="0 0 0" rpy="0 0 0"/>
                 <geometry>
-                    <mesh filename="file://$(find articubot_one)/meshes/${model}.stl" />
+                    <mesh filename="file://$(find blockbuster_core)/meshes/${model}.stl" />
                 </geometry>
                 <material name="mat">

File: description/depthai_macro.urdf.xacro (robot description, xacro)
@@ -5,5 +5,5 @@
                                            cam_pos_x cam_pos_y cam_pos_z
                                            cam_roll cam_pitch cam_yaw r:=0.8 g:=0.8 b:=0.8 a:=0.8 ">
-        <xacro:include filename="$(find articubot_one)/description/base_macro.urdf.xacro"/>
+        <xacro:include filename="$(find blockbuster_core)/description/base_macro.urdf.xacro"/>
         <xacro:property name="M_PI" value="3.1415926535897931" />
         <xacro:property name="model" value="${camera_model}" />

File: description/robot.urdf.xacro (robot description, xacro)
@@ -11,5 +11,5 @@
         <xacro:include filename="gazebo_control.xacro" />
     </xacro:unless>
-    <xacro:include filename="$(find articubot_one)/description/depthai_macro.urdf.xacro"/>
+    <xacro:include filename="$(find blockbuster_core)/description/depthai_macro.urdf.xacro"/>
     <xacro:depthai_camera camera_name = "oak" parent = "base_link" camera_model = "OAK-D-LITE" base_frame = "oak-d_frame" cam_pos_x = "0.2616" cam_pos_y = "-0.0001" cam_pos_z = "0.20" cam_roll = "0" cam_pitch = "0.349" cam_yaw = "0"/>
 </robot>

File: description/robot_core.xacro (robot description, xacro)
@@ -176,5 +176,5 @@
         <origin xyz="-0.104 0.0 -0.2005" rpy="0 0 0"/>
         <geometry>
-        <mesh filename="file://$(find articubot_one)/meshes/Lidar_1.stl" scale="0.001 0.001 0.001"/>
+        <mesh filename="file://$(find blockbuster_core)/meshes/Lidar_1.stl" scale="0.001 0.001 0.001"/>
         </geometry>
         <material name="silver"/>
@@ -183,5 +183,5 @@
         <origin xyz="-0.104 0.0 -0.2005" rpy="0 0 0"/>
         <geometry>
-        <mesh filename="file://$(find articubot_one)/meshes/Lidar_1.stl" scale="0.001 0.001 0.001"/>
+        <mesh filename="file://$(find blockbuster_core)/meshes/Lidar_1.stl" scale="0.001 0.001 0.001"/>
         </geometry>
     </collision>
@@ -196,5 +196,5 @@
         <origin xyz="-0.236 -0.003 -0.208" rpy="0 0 0"/>
         <geometry>
-        <mesh filename="file://$(find articubot_one)/meshes/Stereo_Cam_v1_1.stl" scale="0.001 0.001 0.001"/>
+        <mesh filename="file://$(find blockbuster_core)/meshes/Stereo_Cam_v1_1.stl" scale="0.001 0.001 0.001"/>
         </geometry>
         <material name="silver"/>
@@ -203,5 +203,5 @@
         <origin xyz="-0.236 -0.003 -0.208" rpy="0 0 0"/>
         <geometry>
-        <mesh filename="file://$(find articubot_one)/meshes/Stereo_Cam_v1_1.stl" scale="0.001 0.001 0.001"/>
+        <mesh filename="file://$(find blockbuster_core)/meshes/Stereo_Cam_v1_1.stl" scale="0.001 0.001 0.001"/>
         </geometry>
     </collision>
@@ -216,5 +216,5 @@
         <origin xyz="-0.2616 0.0001 -0.208539" rpy="0 0 0"/>
         <geometry>
-        <mesh filename="file://$(find articubot_one)/meshes/Cam_Window_v1_1.stl" scale="0.001 0.001 0.001"/>
+        <mesh filename="file://$(find blockbuster_core)/meshes/Cam_Window_v1_1.stl" scale="0.001 0.001 0.001"/>
         </geometry>
         <material name="silver"/>
@@ -223,5 +223,5 @@
         <origin xyz="-0.2616 0.0001 -0.208539" rpy="0 0 0"/>
         <geometry>
-        <mesh filename="file://$(find articubot_one)/meshes/Cam_Window_v1_1.stl" scale="0.001 0.001 0.001"/>
+        <mesh filename="file://$(find blockbuster_core)/meshes/Cam_Window_v1_1.stl" scale="0.001 0.001 0.001"/>
         </geometry>
     </collision>

File: description/ros2_control.xacro (robot description, xacro)
@@ -93,6 +93,6 @@
     <gazebo>
         <plugin name="gazebo_ros2_control" filename="libgazebo_ros2_control.so">
-            <parameters>$(find articubot_one)/config/my_controllers.yaml</parameters>
-            <parameters>$(find articubot_one)/config/gaz_ros2_ctl_use_sim.yaml</parameters>
+            <parameters>$(find blockbuster_core)/config/my_controllers.yaml</parameters>
+            <parameters>$(find blockbuster_core)/config/gaz_ros2_ctl_use_sim.yaml</parameters>
         </plugin>
     </gazebo>

File: description/urdf_blockbuster.xacro (robot description, xacro)
@@ -68,5 +68,5 @@
     <origin xyz="0 0 0" rpy="0 0 0"/>
     <geometry>
-      <mesh filename="file://$(find articubot_one)/meshes/base_link.stl" scale="0.001 0.001 0.001"/>
+      <mesh filename="file://$(find blockbuster_core)/meshes/base_link.stl" scale="0.001 0.001 0.001"/>
     </geometry>
   </visual>
@@ -74,5 +74,5 @@
     <origin xyz="0 0 0" rpy="0 0 0"/>
     <geometry>
-      <mesh filename="file://$(find articubot_one)/meshes/base_link.stl" scale="0.001 0.001 0.001"/>
+      <mesh filename="file://$(find blockbuster_core)/meshes/base_link.stl" scale="0.001 0.001 0.001"/>
     </geometry>
   </collision>
@@ -92,5 +92,5 @@
     <origin xyz="0.0575 0.136 -0.03775" rpy="0 0 0"/>
     <geometry>
-      <mesh filename="file://$(find articubot_one)/meshes/Storage_1.stl" scale="0.001 0.001 0.001"/>
+      <mesh filename="file://$(find blockbuster_core)/meshes/Storage_1.stl" scale="0.001 0.001 0.001"/>
     </geometry>
     <material name="silver"/>
@@ -99,5 +99,5 @@
     <origin xyz="0.0575 0.136 -0.03775" rpy="0 0 0"/>
     <geometry>
-      <mesh filename="file://$(find articubot_one)/meshes/Storage_1.stl" scale="0.001 0.001 0.001"/>
+      <mesh filename="file://$(find blockbuster_core)/meshes/Storage_1.stl" scale="0.001 0.001 0.001"/>
     </geometry>
   </collision>
@@ -159,5 +159,5 @@
     <origin xyz="0.243 -0.185 -0.04975" rpy="0 0 0"/>
     <geometry>
-      <mesh filename="file://$(find articubot_one)/meshes/Left_Caster_Wheel_1.stl" scale="0.001 0.001 0.001"/>
+      <mesh filename="file://$(find blockbuster_core)/meshes/Left_Caster_Wheel_1.stl" scale="0.001 0.001 0.001"/>
     </geometry>
     <material name="silver"/>
@@ -166,5 +166,5 @@
     <origin xyz="0.243 -0.185 -0.04975" rpy="0 0 0"/>
     <geometry>
-      <mesh filename="file://$(find articubot_one)/meshes/Left_Caster_Wheel_1.stl" scale="0.001 0.001 0.001"/>
+      <mesh filename="file://$(find blockbuster_core)/meshes/Left_Caster_Wheel_1.stl" scale="0.001 0.001 0.001"/>
     </geometry>
   </collision>
@@ -184,5 +184,5 @@
     <origin xyz="0.243 0.185 -0.04975" rpy="0 0 0"/>
     <geometry>
-      <mesh filename="file://$(find articubot_one)/meshes/Right_Caster_Wheel_1.stl" scale="0.001 0.001 0.001"/>
+      <mesh filename="file://$(find blockbuster_core)/meshes/Right_Caster_Wheel_1.stl" scale="0.001 0.001 0.001"/>
     </geometry>
     <material name="silver"/>
@@ -191,5 +191,5 @@
     <origin xyz="0.243 0.185 -0.04975" rpy="0 0 0"/>
     <geometry>
-      <mesh filename="file://$(find articubot_one)/meshes/Right_Caster_Wheel_1.stl" scale="0.001 0.001 0.001"/>
+      <mesh filename="file://$(find blockbuster_core)/meshes/Right_Caster_Wheel_1.stl" scale="0.001 0.001 0.001"/>
     </geometry>
   </collision>
@@ -209,5 +209,5 @@
     <origin xyz="-0.104 0.0 -0.2005" rpy="0 0 0"/>
     <geometry>
-      <mesh filename="file://$(find articubot_one)/meshes/Lidar_1.stl" scale="0.001 0.001 0.001"/>
+      <mesh filename="file://$(find blockbuster_core)/meshes/Lidar_1.stl" scale="0.001 0.001 0.001"/>
     </geometry>
     <material name="silver"/>
@@ -216,5 +216,5 @@
     <origin xyz="-0.104 0.0 -0.2005" rpy="0 0 0"/>
     <geometry>
-      <mesh filename="file://$(find articubot_one)/meshes/Lidar_1.stl" scale="0.001 0.001 0.001"/>
+      <mesh filename="file://$(find blockbuster_core)/meshes/Lidar_1.stl" scale="0.001 0.001 0.001"/>
     </geometry>
   </collision>
