Commit message: fix: fix of nav2 params & light urdf

File: description/robot.urdf.xacro (robot description, xacro)
@@ -3,6 +3,6 @@
     <xacro:arg name="use_ros2_control" default="true"/>
     <xacro:arg name="sim_mode" default="false"/>
-    <!-- <xacro:include filename="robot_core.xacro" /> -->
-    <xacro:include filename="urdf_blockbuster.xacro" />
+    <xacro:include filename="robot_core.xacro" />
+    <!-- <xacro:include filename="urdf_blockbuster.xacro" /> -->
     <xacro:if value="$(arg use_ros2_control)">
         <xacro:include filename="ros2_control.xacro" />
@@ -12,4 +12,4 @@
     </xacro:unless>
     <xacro:include filename="$(find articubot_one)/description/depthai_macro.urdf.xacro"/>
-    <xacro:depthai_camera camera_name = "oak" parent = "base_link" camera_model = "OAK-D-LITE" base_frame = "oak-d_frame" cam_pos_x = "0.2616" cam_pos_y = "-0.0001" cam_pos_z = "0.20" cam_roll = "0" cam_pitch = "0.785" cam_yaw = "0"/>
+    <xacro:depthai_camera camera_name = "oak" parent = "base_link" camera_model = "OAK-D-LITE" base_frame = "oak-d_frame" cam_pos_x = "0.2616" cam_pos_y = "-0.0001" cam_pos_z = "0.20" cam_roll = "0" cam_pitch = "0.524" cam_yaw = "0"/>
 </robot>

File: description/robot_core.xacro (robot description, xacro)
@@ -233,5 +233,5 @@
     </joint>
     <joint name="Stereo Cam" type="fixed">
-        <origin xyz="0.236 0.003 0.208" rpy="0 0.785 0"/>
+        <origin xyz="0.236 0.003 0.208" rpy="0 0.524 0"/>
         <parent link="base_link"/>
         <child link="Stereo_Cam_v1_1"/>
@@ -242,4 +242,25 @@
         <child link="Cam_Window_v1_1"/>
     </joint>
+    <joint name="storage_joint" type="continuous">
+        <origin xyz="-0.20 0.13 0.13" rpy="1.57 0 0"/>
+        <parent link="base_link"/>
+        <child link="servo_frame"/>
+    </joint>
+    <link name="servo_frame">
+        <visual>
+            <geometry>
+                <cylinder radius="0.01" length="0.005"/>
+            </geometry>
+        </visual>
+        <collision>
+            <geometry>
+                <sphere radius="0.051"/>
+            </geometry>
+        </collision>
+        <inertial>
+            <mass value="0.04021467988426049"/>
+            <inertia ixx="4e-05" iyy="7e-05" izz="4e-05" ixy="-0.0" iyz="0.0" ixz="0.0"/>
+        </inertial>
+    </link>
     <gazebo reference="laser_frame">
         <material>Gazebo/Black</material>

Commit message: fix: fix for hardware robot

File: description/robot.urdf.xacro (robot description, xacro)
@@ -12,4 +12,4 @@
     </xacro:unless>
     <xacro:include filename="$(find articubot_one)/description/depthai_macro.urdf.xacro"/>
-    <xacro:depthai_camera camera_name = "oak" parent = "base_link" camera_model = "OAK-D-LITE" base_frame = "oak-d_frame" cam_pos_x = "0.2616" cam_pos_y = "-0.0001" cam_pos_z = "0.20" cam_roll = "0" cam_pitch = "0.524" cam_yaw = "0"/>
+    <xacro:depthai_camera camera_name = "oak" parent = "base_link" camera_model = "OAK-D-LITE" base_frame = "oak-d_frame" cam_pos_x = "0.2616" cam_pos_y = "-0.0001" cam_pos_z = "0.20" cam_roll = "0" cam_pitch = "0.349" cam_yaw = "0"/>
 </robot>

File: description/robot_core.xacro (robot description, xacro)
@@ -233,5 +233,5 @@
     </joint>
     <joint name="Stereo Cam" type="fixed">
-        <origin xyz="0.236 0.003 0.208" rpy="0 0.524 0"/>
+        <origin xyz="0.236 0.003 0.208" rpy="0 0.349 0"/>
         <parent link="base_link"/>
         <child link="Stereo_Cam_v1_1"/>

Commit message: fix: fixes after arena testing M1

File: description/robot.urdf.xacro (robot description, xacro)
@@ -12,4 +12,4 @@
     </xacro:unless>
     <xacro:include filename="$(find blockbuster_core)/description/depthai_macro.urdf.xacro"/>
-    <xacro:depthai_camera camera_name = "oak" parent = "base_link" camera_model = "OAK-D-LITE" base_frame = "oak-d_frame" cam_pos_x = "0.2616" cam_pos_y = "-0.0001" cam_pos_z = "0.20" cam_roll = "0" cam_pitch = "0.349" cam_yaw = "0"/>
+    <xacro:depthai_camera camera_name = "oak" parent = "base_link" camera_model = "OAK-D-LITE" base_frame = "oak-d_frame" cam_pos_x = "0.2616" cam_pos_y = "-0.0001" cam_pos_z = "0.20" cam_roll = "0" cam_pitch = "0.175" cam_yaw = "0"/>
 </robot>

File: description/robot_core.xacro (robot description, xacro)
@@ -233,5 +233,5 @@
     </joint>
     <joint name="Stereo Cam" type="fixed">
-        <origin xyz="0.236 0.003 0.208" rpy="0 0.349 0"/>
+        <origin xyz="0.236 0.003 0.208" rpy="0 0.175 0"/>
         <parent link="base_link"/>
         <child link="Stereo_Cam_v1_1"/>

File: description/ros2_control.xacro (robot description, xacro)
@@ -20,6 +20,6 @@
             <joint name="left_wheel_joint">
                 <command_interface name="velocity">
-                    <param name="min">-10</param>
-                    <param name="max">10</param>
+                    <param name="min">-20</param>
+                    <param name="max">20</param>
                 </command_interface>
                 <state_interface name="position"/>
@@ -28,6 +28,6 @@
             <joint name="right_wheel_joint">
                 <command_interface name="velocity">
-                    <param name="min">-10</param>
-                    <param name="max">10</param>
+                    <param name="min">-20</param>
+                    <param name="max">20</param>
                 </command_interface>
                 <state_interface name="position"/>
